File: BQ25798.kicad_pcb (KiCad board)
At the start: 2 copper layers, 30.5 x 35.6 mm, 45 parts, among them J1 VIN, J2 SYS_OUT, J3 BATTERY, J4 I2C, U1 BQ25798

Commit message: Completed PCB
Parts:
- moved C9 2.21 mm to (136.2, 84.5)
- turned C15 to 0 degrees
Routing:
- net SYS: track 0.00 -> 79.4 mm, vias 0 -> 4
- net SCL: track 0.00 -> 75.4 mm, vias 0 -> 10
- net SDA: track 0.00 -> 73.7 mm, vias 0 -> 6
- net INT: track 0.00 -> 67.1 mm
- net CE: track 0.00 -> 61.9 mm, vias 0 -> 10
- net QON: track 0.00 -> 54.9 mm, vias 0 -> 2
- net GND: track 0.37 -> 55.0 mm, vias 0 -> 11
- net Net-(U1-SW2): track 1.28 -> 41.6 mm, vias 0 -> 4
- net TS: track 0.00 -> 34.6 mm, vias 0 -> 2
- net Net-(J1-Pin_1): track 0.00 -> 33.1 mm, vias 0 -> 3
- net REGN: track 0.00 -> 27.9 mm, vias 0 -> 2
- net ILIM_HIZ: track 0.00 -> 24.5 mm, vias 0 -> 2
- net BAT: track 0.69 -> 20.6 mm, vias 0 -> 2
- net Net-(U1-SW1): track 0.00 -> 18.8 mm, vias 0 -> 2
- net STAT: track 0.00 -> 16.4 mm, vias 0 -> 2
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- added copper zone on B.Cu, net GND
